Commit message: Problema solucionado .xacro

File: urdf/Kwad.xacro (robot description, xacro)
@@ -11,6 +11,6 @@
 	<xacro:property name="prop_loc" value="0.15909" />
 <!-- ======================================================== -->
-	<xacro:include filename="$(find fly_bot)/urdf/material.xacro" />
-	<xacro:include filename="$(find fly_bot)/urdf/Kwad.gazebo" />
+	<xacro:include filename="$(find first_version_proj)/urdf/material.xacro" />
+	<xacro:include filename="$(find first_version_proj)/urdf/Kwad.gazebo" />
 <!-- ======================================================== -->
 	<!-- Define inertial macro -->
@@ -164,5 +164,5 @@
 			<origin xyz="0 0 0" rpy="0 0 0" />
 			<geometry>
-				<mesh filename="package://fly_bot/meshes/22V10.dae" scale="0.005 0.005 0.005" />
+				<mesh filename="package://first_version_proj/meshes/22V10.dae" scale="0.005 0.005 0.005" />
 			</geometry>
 		</visual>
