Commit message: Cambio a drone parrot

File: urdf/Obstacle1.urdf (robot description, URDF)
Before this commit: robot robot_name, 3 links, 2 joints
Links:
- link base_link: mass 1.0 -> 10.0
- link obst: mass 1.0 -> 10.0
Joints:
- joint joint_mov: limit lower=-0.5 upper=1 effort=300 velocity=1 -> lower=-1 upper=1 effort=300 velocity=1; origin xyz=0 0 1.5 rpy=0 0 0 -> xyz=0 0 2 rpy=0 0 0
