Commit message: Se agregaron sensores

File: urdf/parrot.xacro (robot description, xacro)
@@ -25,5 +25,6 @@
 <!-- ======================================================== -->
 	<link name="base_link1">
-        <origin xyz="0 0 0" rpy="0 0 ${pi_value/4}" />
+        <!--origin xyz="0 0 0" rpy="0 0 ${pi_value/4}" /-->
+		<origin xyz="0 0 0" rpy="0 0 0" />
 		<visual>
 			<origin xyz="0 0 0" rpy="0 0 0" />
@@ -105,4 +106,45 @@
 		<xacro:default_inertial mass="${mass_pr}" p="${0}"  ix_value="${0}" iy_value="${0}" iz_value="${4.42448e-5}" />
 	</link>
+	<link name="vertical_camera_link">
+		<visual>
+			<origin xyz="0 0 0" rpy="0 0 0" />
+			<geometry>
+				<box size="0.002 0.01 0.005" />
+			</geometry>
+			<material name="red" />
+		</visual>
+		<collision>
+			<origin xyz="0 0 0" rpy="0 0 0" />
+			<geometry>
+				<box size="0.01 0.01 0.005" />
+			</geometry>
+		</collision>
+		<xacro:default_inertial mass="${1e-5}" p="${0}" ix_value="${1e-6}" iy_value="${1e-6}" iz_value="${1e-6}" />
+	</link>
+	<link name="front_camera_link">
+		<visual>
+			<origin xyz="0 0 0" rpy="0 0 0" />
+			<geometry>
+				<box size="0.002 0.05 0.05" />
+			</geometry>
+			<material name="red" />
+		</visual>
+		<collision>
+			<origin xyz="0 0 0" rpy="0 0 0" />
+			<geometry>
+				<box size="0.002 0.05 0.05" />
+			</geometry>
+		</collision>
+		<xacro:default_inertial mass="${1e-5}" p="${0}" ix_value="${1e-6}" iy_value="${1e-6}" iz_value="${1e-6}" />
+	</link>
+    <link name="gyro_link">
+      <inertial>
+        <mass value="0.001"/>
+        <origin xyz="0 0 0" rpy="0 0 0"/>
+        <inertia ixx="0.0001" ixy="0" ixz="0"
+                 iyy="0.000001" iyz="0"
+                 izz="0.0001"/>
+      </inertial>
+    </link>
     <joint name="joint_front_right_prop" type="continuous">
 		<parent link="base_link1" />
@@ -134,4 +176,22 @@
 		<axis xyz="0 0 1" />
 	</joint>
+	<joint name="joint_vertical_camera_frame" type="fixed">
+		<parent link="base_link1" />
+		<child link="vertical_camera_link" />
+		<origin xyz="0.0 0.0 -0.008" rpy="0 ${pi_value/2} 0" />
+		<axis xyz="0 0 1" />
+	</joint>
+	<joint name="joint_front_camera_frame" type="fixed">
+		<parent link="base_link1" />
+		<child link="front_camera_link" />
+		<origin xyz="0.2921 0.0 0.0" rpy="0 0 0" />
+		<axis xyz="1 0 0" />
+	</joint>
+	<joint name="gyro_joint" type="fixed">
+      <axis xyz="0 0 1"/>
+      <origin xyz="0.0 0.0 0.0202" rpy="0 0 0"/>
+      <parent link="base_link1"/>
+      <child link="gyro_link"/>
+    </joint>
     <transmission name="front_right_motor_joint" >
 		<type>transmission_interface/SimpleTransmission</type>
